Commit message: added d435 urdf

File: autovalet_description/urdf/husky.urdf.xacro (robot description, xacro)
@@ -40,4 +40,6 @@
   <!-- Subbu: Included VLP-16 xacro file from another package here-->
   <xacro:include filename="$(find autovalet_description)/urdf/accessories/VLP-16.urdf.xacro"/>
+  <!-- Subbu: Inculded d435 xacro file from realsense2 official description-->
+  <xacro:include filename="$(find autovalet_description)/urdf/accessories/_d435.urdf.xacro"/>
   <xacro:property name="M_PI" value="3.14159"/>
   <!-- Base Size -->
@@ -141,4 +143,7 @@
     <origin xyz="0 0 0.4" rpy="0 0 0" />
   </VLP-16>
+  <sensor_d435 parent="base_link" name="d435_frontCamera" >
+    <origin xyz="0 0 0.7" rpy="0 0 0" />
+  </sensor_d435>
   <gazebo>
     <plugin name="gazebo_ros_control" filename="libgazebo_ros_control.so">
