Commit message: updated joystick config in valet_husky

File: autovalet_description/urdf/autovalet.urdf.xacro (robot description, xacro)
@@ -6,14 +6,14 @@
 	<xacro:include filename="$(find velodyne_description)/urdf/VLP-16.urdf.xacro"/>
 	<!-- Define the front camera link -->
-	<sensor_d435 parent="top_plate_link" name="frontCamera" >
-	    <origin xyz="0.35 0 0.005" rpy="0 0 0" />
+	<sensor_d435 parent="velodyne" name="backCamera" >
+	    <origin xyz="0 -0.11 -0.05" rpy="0 0 -1.57079" />
 	</sensor_d435>
 	<!-- Define the back camera link -->
-	<sensor_d435 parent="top_plate_link" name="backCamera" >
-	    <origin xyz="-0.35 0 0.005" rpy="0 0 3.1415"/>
+	<sensor_d435 parent="velodyne" name="frontCamera" >
+	    <origin xyz="0 0.197 -0.05" rpy="0 0 1.57079"/>
 	</sensor_d435>
 	<!-- Define the velodyne link to the husky -->
-	<VLP-16 parent="top_plate_link" name="velodyne" topic="/velodyne_points" hz="10" samples="440">
-    	<origin xyz="0 0 0.005" rpy="0 0 0"/>
+	<VLP-16 parent="base_link" name="velodyne" topic="/velodyne_points" hz="10" samples="440">
+    	<origin xyz="0 -0.015 0.345" rpy="0 0 -1.570796326"/>
   	</VLP-16>
 </robot>

Commit message: updated urdf to have sensor placements for a ford focus

File: autovalet_description/urdf/autovalet.urdf.xacro (robot description, xacro)
@@ -7,13 +7,13 @@
 	<!-- Define the front camera link -->
 	<sensor_d435 parent="velodyne" name="backCamera" >
-	    <origin xyz="0 -0.11 -0.05" rpy="0 0 -1.57079" />
+	    <origin xyz="0 -0.11 -0.59" rpy="0 0 -1.57079" />
 	</sensor_d435>
 	<!-- Define the back camera link -->
 	<sensor_d435 parent="velodyne" name="frontCamera" >
-	    <origin xyz="0 0.197 -0.05" rpy="0 0 1.57079"/>
+	    <origin xyz="0 0.197 -0.59" rpy="0 0 1.57079"/>
 	</sensor_d435>
-	<!-- Define the velodyne link to the husky -->
-	<VLP-16 parent="base_link" name="velodyne" topic="/velodyne_points" hz="10" samples="440">
-    	<origin xyz="0 -0.015 0.345" rpy="0 0 -1.570796326"/>
+	<!-- Define the velodyne link to the husky (base_link)-->
+	<VLP-16 parent="base_footprint" name="velodyne" topic="/velodyne_points" hz="10" samples="440">
+    	<origin xyz="0 -0.015 1.47" rpy="0 0 -1.570796326"/>
   	</VLP-16>
 </robot>

Commit message: camera extrinsic modified
added the tf between lidar and camera using manual calib tool

cam param config

enhance camera resolution to color-1920x1080, depth-848x480

File: autovalet_description/urdf/autovalet.urdf.xacro (robot description, xacro)
@@ -5,15 +5,15 @@
 	<!-- Include the velodyne model from the velodyne description package-->
 	<xacro:include filename="$(find velodyne_description)/urdf/VLP-16.urdf.xacro"/>
-	<!-- Define the front camera link -->
-	<sensor_d435 parent="velodyne" name="backCamera" >
-	    <origin xyz="0 -0.11 -0.59" rpy="0 0 -1.57079" />
+	<sensor_d435 parent="front_bumper_link" name="frontCamera" >
+	    <origin xyz="-0.305 0.02 0.91" rpy="0 0 0" />
 	</sensor_d435>
-	<!-- Define the back camera link -->
-	<sensor_d435 parent="velodyne" name="frontCamera" >
-	    <origin xyz="0 0.197 -0.59" rpy="0 0 1.57079"/>
+	<!-- Define the back camera link to the front camera-->
+	<sensor_d435 parent="frontCamera_bottom_screw_frame" name="backCamera" >
+	    <origin xyz="-0.235 0 0" rpy="0 0 3.14159"/>
 	</sensor_d435>
-	<!-- Define the velodyne link to the husky (base_link)-->
-	<VLP-16 parent="base_footprint" name="velodyne" topic="/velodyne_points" hz="10" samples="440">
-    	<origin xyz="0 -0.015 1.47" rpy="0 0 -1.570796326"/>
+	<!-- Define the velodyne link to the front camera-->
+	<VLP-16 parent="frontCamera_bottom_screw_frame" name="velodyne" topic="/velodyne_points" hz="10" samples="440">
+        <!-- the z coordinate is wrong. in our sensor frame, it's more like .35m. but .22m aligns the point clouds in rviz...-->
+    	<origin xyz="-0.155 0.0 0.22" rpy="0.0 0.0 0.0"/>
   	</VLP-16>
 </robot>

Commit message: left turns with intermediate goals

File: autovalet_description/urdf/autovalet.urdf.xacro (robot description, xacro)
@@ -6,5 +6,5 @@
 	<xacro:include filename="$(find velodyne_description)/urdf/VLP-16.urdf.xacro"/>
 	<sensor_d435 parent="front_bumper_link" name="frontCamera" >
-	    <origin xyz="-0.305 0.02 0.91" rpy="0 0 0" />
+	    <origin xyz="-0.305 0.02 0.91" rpy="0 0.174 0" />
 	</sensor_d435>
 	<!-- Define the back camera link to the front camera-->
@@ -15,5 +15,5 @@
 	<VLP-16 parent="frontCamera_bottom_screw_frame" name="velodyne" topic="/velodyne_points" hz="10" samples="440">
         <!-- the z coordinate is wrong. in our sensor frame, it's more like .35m. but .22m aligns the point clouds in rviz...-->
-    	<origin xyz="-0.155 0.0 0.22" rpy="0.0 0.0 0.0"/>
+    	<origin xyz="-0.155 0.0 0.22" rpy="0.0 -0.174 0.0"/>
   	</VLP-16>
 </robot>

Commit message: Lot testing final tweaks

File: autovalet_description/urdf/autovalet.urdf.xacro (robot description, xacro)
@@ -6,5 +6,9 @@
 	<xacro:include filename="$(find velodyne_description)/urdf/VLP-16.urdf.xacro"/>
 	<sensor_d435 parent="front_bumper_link" name="frontCamera" >
-	    <origin xyz="-0.305 0.02 0.91" rpy="0 0.174 0" />
+	    <!-- Reduced camera hight -->
+		<origin xyz="-0.305 0.02 0.71" rpy="0 0.0 0" />
+		<!-- The standard one for H/w -->
+		<!-- <origin xyz="-0.305 0.02 0.91" rpy="0 0.0 0" /> -->
+		<!-- <origin xyz="-0.305 0.02 0.91" rpy="0 0.174 0" /> -->
 	</sensor_d435>
 	<!-- Define the back camera link to the front camera-->
@@ -15,5 +19,9 @@
 	<VLP-16 parent="frontCamera_bottom_screw_frame" name="velodyne" topic="/velodyne_points" hz="10" samples="440">
         <!-- the z coordinate is wrong. in our sensor frame, it's more like .35m. but .22m aligns the point clouds in rviz...-->
-    	<origin xyz="-0.155 0.0 0.22" rpy="0.0 -0.174 0.0"/>
+		<!-- Reduced camera height -->
+		<origin xyz="-0.155 0.0 0.42" rpy="0.0 0.0 0.0"/>
+		<!-- Standard position for lidar -->
+		<!-- <origin xyz="-0.155 0.0 0.22" rpy="0.0 0.0 0.0"/> -->
+		<!-- <origin xyz="-0.155 0.0 0.22" rpy="0.0 -0.174 0.0"/> -->
   	</VLP-16>
 </robot>

Commit message: urdf corrected

File: autovalet_description/urdf/autovalet.urdf.xacro (robot description, xacro)
@@ -6,5 +6,6 @@
 	<xacro:include filename="$(find velodyne_description)/urdf/VLP-16.urdf.xacro"/>
 	<sensor_d435 parent="front_bumper_link" name="frontCamera" >
-	    <origin xyz="-0.305 0.02 0.91" rpy="0 0.174 0" />
+	    <origin xyz="-0.305 0.02 0.91" rpy="0 0.0 0" />
+		<!-- <origin xyz="-0.305 0.02 0.91" rpy="0 0.174 0" /> -->
 	</sensor_d435>
 	<!-- Define the back camera link to the front camera-->
@@ -15,5 +16,6 @@
 	<VLP-16 parent="frontCamera_bottom_screw_frame" name="velodyne" topic="/velodyne_points" hz="10" samples="440">
         <!-- the z coordinate is wrong. in our sensor frame, it's more like .35m. but .22m aligns the point clouds in rviz...-->
-    	<origin xyz="-0.155 0.0 0.22" rpy="0.0 -0.174 0.0"/>
+    	<origin xyz="-0.155 0.0 0.22" rpy="0.0 0.0 0.0"/>
+		<!-- <origin xyz="-0.155 0.0 0.22" rpy="0.0 -0.174 0.0"/> -->
   	</VLP-16>
 </robot>

Commit message: two right turns working

File: autovalet_description/urdf/autovalet.urdf.xacro (robot description, xacro)
@@ -6,5 +6,8 @@
 	<xacro:include filename="$(find velodyne_description)/urdf/VLP-16.urdf.xacro"/>
 	<sensor_d435 parent="front_bumper_link" name="frontCamera" >
-	    <origin xyz="-0.305 0.02 0.91" rpy="0 0.0 0" />
+	    <!-- Reduced camera hight -->
+		<origin xyz="-0.305 0.02 0.71" rpy="0 0.0 0" />
+		<!-- The standard one for H/w -->
+		<!-- <origin xyz="-0.305 0.02 0.91" rpy="0 0.0 0" /> -->
 		<!-- <origin xyz="-0.305 0.02 0.91" rpy="0 0.174 0" /> -->
 	</sensor_d435>
@@ -16,5 +19,8 @@
 	<VLP-16 parent="frontCamera_bottom_screw_frame" name="velodyne" topic="/velodyne_points" hz="10" samples="440">
         <!-- the z coordinate is wrong. in our sensor frame, it's more like .35m. but .22m aligns the point clouds in rviz...-->
-    	<origin xyz="-0.155 0.0 0.22" rpy="0.0 0.0 0.0"/>
+		<!-- Reduced camera height -->
+		<origin xyz="-0.155 0.0 0.42" rpy="0.0 0.0 0.0"/>
+		<!-- Standard position for lidar -->
+		<!-- <origin xyz="-0.155 0.0 0.22" rpy="0.0 0.0 0.0"/> -->
 		<!-- <origin xyz="-0.155 0.0 0.22" rpy="0.0 -0.174 0.0"/> -->
   	</VLP-16>
