Commit message: plugin functionality added

File: autovalet_realsense/realsense2_description/urdf/_d435.urdf.xacro (robot description, xacro)
@@ -13,5 +13,5 @@
   <!-- For running with gazebo sim -->
   <xacro:arg name="use_nominal_extrinsics" default="false"/>
-  <xacro:macro name="sensor_d435" params="parent *origin name:=camera">
+  <xacro:macro name="sensor_d435" params="parent *origin name:=camera topics_ns:=realsense">
     <xacro:property name="M_PI" value="3.1415926535897931" />
     <!-- The following values are approximate, and the camera node
@@ -119,5 +119,5 @@
       </joint>
       <link name="${name}_color_optical_frame"/>
-      <!-- <xacro:gazebo_d435 camera_name="${name}" reference_link="${name}_link" topics_ns="${topics_ns}" depth_optical_frame="${name}_depth_optical_frame" color_optical_frame="${name}_color_optical_frame" infrared1_optical_frame="${name}_left_ir_optical_frame" infrared2_optical_frame="${name}_right_ir_optical_frame"/> -->
+      <xacro:gazebo_d435 camera_name="${name}" reference_link="${name}_link" topics_ns="${topics_ns}" depth_optical_frame="${name}_depth_optical_frame" color_optical_frame="${name}_color_optical_frame" infrared1_optical_frame="${name}_left_ir_optical_frame" infrared2_optical_frame="${name}_right_ir_optical_frame"/>
     </xacro:if>
   </xacro:macro>

File: autovalet_realsense/realsense_gazebo_plugin/urdf/realsense.gazebo.xacro (robot description, xacro)
@@ -114,15 +114,15 @@
       <plugin name="${topics_ns}" filename="librealsense_gazebo_plugin.so">
         <prefix>${camera_name}</prefix>
-      	<depthUpdateRate>60.0</depthUpdateRate>
-      	<colorUpdateRate>60.0</colorUpdateRate>
+      	<depthUpdateRate>100.0</depthUpdateRate>
+      	<colorUpdateRate>100.0</colorUpdateRate>
       	<infraredUpdateRate>60.0</infraredUpdateRate>
-      	<depthTopicName>depth/image_raw</depthTopicName>
-      	<depthCameraInfoTopicName>depth/camera_info</depthCameraInfoTopicName>
-      	<colorTopicName>color/image_raw</colorTopicName>
-      	<colorCameraInfoTopicName>color/camera_info</colorCameraInfoTopicName>
-      	<infrared1TopicName>infra1/image_raw</infrared1TopicName>
-      	<infrared1CameraInfoTopicName>infra1/camera_info</infrared1CameraInfoTopicName>
-      	<infrared2TopicName>infra2/image_raw</infrared2TopicName>
-      	<infrared2CameraInfoTopicName>infra2/camera_info</infrared2CameraInfoTopicName>
+      	<depthTopicName>${camera_name}/depth/image_raw</depthTopicName>
+      	<depthCameraInfoTopicName>${camera_name}/depth/camera_info</depthCameraInfoTopicName>
+      	<colorTopicName>${camera_name}/color/image_raw</colorTopicName>
+      	<colorCameraInfoTopicName>${camera_name}/color/camera_info</colorCameraInfoTopicName>
+      	<infrared1TopicName>${camera_name}/infra1/image_raw</infrared1TopicName>
+      	<infrared1CameraInfoTopicName>${camera_name}/infra1/camera_info</infrared1CameraInfoTopicName>
+      	<infrared2TopicName>${camera_name}/infra2/image_raw</infrared2TopicName>
+      	<infrared2CameraInfoTopicName>${camera_name}/infra2/camera_info</infrared2CameraInfoTopicName>
       	<colorOpticalframeName>${color_optical_frame}</colorOpticalframeName>
       	<depthOpticalframeName>${depth_optical_frame}</depthOpticalframeName>
@@ -131,6 +131,6 @@
       	<rangeMinDepth>0.2</rangeMinDepth>
       	<rangeMaxDepth>10.0</rangeMaxDepth>
-      	<pointCloud>false</pointCloud>
-      	<pointCloudTopicName>depth/points</pointCloudTopicName>
+      	<pointCloud>true</pointCloud>
+      	<pointCloudTopicName>${camera_name}/depth/points</pointCloudTopicName>
       	<pointCloudCutoff>0.5</pointCloudCutoff>
       </plugin>

File: vlp16_simulator/velodyne_description/urdf/VLP-16.urdf.xacro (robot description, xacro)
@@ -52,5 +52,5 @@
     </link>
     <!-- Gazebo requires the velodyne_gazebo_plugins package -->
-<!--     <gazebo reference="${name}">
+    <gazebo reference="${name}">
       <xacro:if value="${gpu}">
         <sensor type="gpu_ray" name="${name}-VLP16">
@@ -133,5 +133,5 @@
         </sensor>
       </xacro:unless>
-    </gazebo> -->
+    </gazebo>
   </xacro:macro>
 </robot>

Commit message: Changed the ground plane to be artificially green Added online segmentation map generating script
Added the goal generation package
Corrected the namespace for realsense in simulation

Added lane segmentation in cloud

Added the goal generation package
Corrected the namespace for realsense in simulation

Added lane segmentation in cloud

Added lane segmenter in cloud to project the segmented depth map of the lane back onto the real world
Added a fake "lane" sensor in the costmap commons params file

/realsense namespace removed
depth image registered to rgb image
lane pcl projected onto constmap
goal transfer launch files created

removed static params yaml and updated global costmap params

removed static map params and updated global cmap params for sim and hw

Changed the ground plane to be artificially green
Added online segmentation map generating script

Added lane segmentation in cloud

segmap uncommented in launch file

File: autovalet_realsense/realsense2_description/urdf/_d435.urdf.xacro (robot description, xacro)
@@ -13,5 +13,5 @@
   <!-- For running with gazebo sim -->
   <xacro:arg name="use_nominal_extrinsics" default="false"/>
-  <xacro:macro name="sensor_d435" params="parent *origin name:=camera topics_ns:=realsense">
+  <xacro:macro name="sensor_d435" params="parent *origin name:=camera topics_ns:=/">
     <xacro:property name="M_PI" value="3.1415926535897931" />
     <!-- The following values are approximate, and the camera node
